Commit message: update for today its working

File: src/notspot_description/urdf/notspot copy.urdf (robot description, URDF)
Before this commit: robot notspot, 25 links, 24 joints
Links:
- removed link end_effector_link
- removed link gripper_link
- removed link gripper_link_sub
- removed link link1
- removed link link2
- removed link link3
- removed link link4
- removed link link5
- added link arm_base_link, mass 0.16646514073208918; collision mesh filename=package://arm_description/meshes/base_link.stl scale=0.001 0.001 0.001; visual mesh filename=package://arm_description/meshes/base_link.stl scale=0.001 0.001 0.001
- added link link_2_1, mass 0.12976814590575328; collision mesh filename=package://arm_description/meshes/link_2_1.stl scale=0.001 0.001 0.001; visual mesh filename=package://arm_description/meshes/link_2_1.stl scale=0.001 0.001 0.001
- added link link_3_1, mass 0.1802231565147444; collision mesh filename=package://arm_description/meshes/link_3_1.stl scale=0.001 0.001 0.001; visual mesh filename=package://arm_description/meshes/link_3_1.stl scale=0.001 0.001 0.001
- added link link_4_1, mass 0.020886761648388527; collision mesh filename=package://arm_description/meshes/link_4_1.stl scale=0.001 0.001 0.001; visual mesh filename=package://arm_description/meshes/link_4_1.stl scale=0.001 0.001 0.001
- added link link_7_1, mass 0.04974076971131721; collision mesh filename=package://arm_description/meshes/link_7_1.stl scale=0.001 0.001 0.001; visual mesh filename=package://arm_description/meshes/link_7_1.stl scale=0.001 0.001 0.001
Joints:
- removed joint end_effector_joint
- removed joint gripper
- removed joint gripper_sub
- removed joint joint1
- removed joint joint2
- removed joint joint3
- removed joint joint4
- removed joint world_fixed
- added joint Rev10: type continuous, parent link_4_1, child link_7_1, origin xyz=0.005004 0.025 -5e-06 rpy=0 0 0, axis -0.0 1.0 -0.0
- added joint Rev7: type continuous, parent arm_base_link, child link_2_1, origin xyz=0.0 0.0 0.03 rpy=0 0 0, axis 0.0 0.0 1.0
- added joint Rev8: type revolute, parent link_2_1, child link_3_1, origin xyz=-0.0 0.028583 0.04309 rpy=0 0 0, axis -1.0 0.0 0.0, limit lower=-0.785398 upper=0.785398 effort=100 velocity=100
- added joint Rev9: type revolute, parent link_3_1, child link_4_1, origin xyz=0.0 0.12 0.0 rpy=0 0 0, axis 1.0 0.0 -0.0, limit lower=-1.570796 upper=0.0 effort=100 velocity=100
- added joint base: type fixed, parent base_link, child arm_base_link, origin xyz=0.1 0.0 0.03 rpy=0 0 0, axis 0.0 0.0 1.0, limit lower=0.0 upper=0.548 effort=1000.0 velocity=0.5
