Commit message: change

File: src/notspot_description/urdf/notspot.urdf (robot description, URDF)
Before this commit: robot notspot, 17 links, 16 joints
Links:
- added link arm_base_link, mass 0.16646514073208918; collision mesh filename=package://arm_description/meshes/base_link.stl scale=0.001 0.001 0.001; visual mesh filename=package://arm_description/meshes/base_link.stl scale=0.001 0.001 0.001
- added link link_2_1, mass 0.12976814590575328; collision mesh filename=package://arm_description/meshes/link_2_1.stl scale=0.001 0.001 0.001; visual mesh filename=package://arm_description/meshes/link_2_1.stl scale=0.001 0.001 0.001
- added link link_3_1, mass 0.1802231565147444; collision mesh filename=package://arm_description/meshes/link_3_1.stl scale=0.001 0.001 0.001; visual mesh filename=package://arm_description/meshes/link_3_1.stl scale=0.001 0.001 0.001
- added link link_4_1, mass 0.020886761648388527; collision mesh filename=package://arm_description/meshes/link_4_1.stl scale=0.001 0.001 0.001; visual mesh filename=package://arm_description/meshes/link_4_1.stl scale=0.001 0.001 0.001
- added link link_7_1, mass 0.04974076971131721; collision mesh filename=package://arm_description/meshes/link_7_1.stl scale=0.001 0.001 0.001; visual mesh filename=package://arm_description/meshes/link_7_1.stl scale=0.001 0.001 0.001
Joints:
- added joint Rev10: type continuous, parent link_4_1, child link_7_1, origin xyz=0.005004 0.025 -5e-06 rpy=0 0 0, axis -0.0 1.0 -0.0
- added joint Rev7: type continuous, parent arm_base_link, child link_2_1, origin xyz=0.0 0.0 0.03 rpy=0 0 0, axis 0.0 0.0 1.0
- added joint Rev8: type revolute, parent link_2_1, child link_3_1, origin xyz=-0.0 0.028583 0.04309 rpy=0 0 0, axis -1.0 0.0 0.0, limit lower=-0.785398 upper=0.785398 effort=100 velocity=100
- added joint Rev9: type revolute, parent link_3_1, child link_4_1, origin xyz=0.0 0.12 0.0 rpy=0 0 0, axis 1.0 0.0 -0.0, limit lower=-1.570796 upper=0.0 effort=100 velocity=100
- added joint base: type fixed, parent base_link, child arm_base_link, origin xyz=0.0 0.0 0.03 rpy=0 0 0, axis 0.0 0.0 1.0, limit lower=0.0 upper=0.548 effort=1000.0 velocity=0.5

Commit message: update for arm base

File: src/notspot_description/urdf/notspot.urdf (robot description, URDF)
Before this commit: robot notspot, 22 links, 21 joints
Joints:
- joint base: origin xyz=0.0 0.0 0.03 rpy=0 0 0 -> xyz=0.1 0.0 0.03 rpy=0 0 0

Commit message: added tray for ford

File: src/notspot_description/urdf/notspot.urdf (robot description, URDF)
Before this commit: robot notspot, 25 links, 24 joints
Links:
- added link tray, mass 0.017; collision mesh filename=package://open_manipulator_description/meshes/tray.stl scale=0.0004 0.0004 0.0004; visual mesh filename=package://open_manipulator_description/meshes/tray.stl scale=0.0004 0.0004 0.0004
Joints:
- added joint joint_tray: type fixed, parent base_link, child tray, origin xyz=-0.08 0.0 -0.095 rpy=0.0 0.0 1.5708, axis 0.0 0.0 0.0
- joint joint1: origin xyz=0.012 0.0 0.017 rpy=0 0 0 -> xyz=0.012 0.0 0.017 rpy=0 0 1.57
