Commit message: complete working

File: src/notspot_description/urdf/materials.xacro (robot description, xacro)
@@ -4,3 +4,30 @@
   <color rgba="0.700 0.700 0.700 1.000"/>
 </material>
+<material name="black">
+  <color rgba="0.0 0.0 0.0 1.0"/>
+</material>
+<material name="white">
+  <color rgba="1.0 1.0 1.0 1.0"/>
+</material>
+<material name="red">
+  <color rgba="0.8 0.0 0.0 1.0"/>
+</material>
+<material name="blue">
+  <color rgba="0.0 0.0 0.8 1.0"/>
+</material>
+<material name="green">
+  <color rgba="0.0 0.8 0.0 1.0"/>
+</material>
+<material name="grey">
+  <color rgba="0.5 0.5 0.5 1.0"/>
+</material>
+<material name="orange">
+  <color rgba="${255/255} ${108/255} ${10/255} 1.0"/>
+</material>
+<material name="brown">
+  <color rgba="${222/255} ${207/255} ${195/255} 1.0"/>
+</material>
+<material name="yellow">
+  <color rgba="${232/255} ${173/255} ${35/255} 1.0"/>
+</material>
 </robot>

File: src/notspot_description/urdf/notspot.urdf (robot description, URDF)
Before this commit: robot notspot, 26 links, 25 joints
Links:
- removed link end_effector_link
- link gripper_link: geometry collision mesh filename=package://notspot_description/meshes/chain_link_grip_l.stl scale=0.001 0.001 0.001; visual mesh filename=package://notspot_description/meshes/chain_link_grip_l.stl scale=0.001 0.001 0.001
- link gripper_link_sub: geometry collision mesh filename=package://notspot_description/meshes/chain_link_grip_r.stl scale=0.001 0.001 0.001; visual mesh filename=package://notspot_description/meshes/chain_link_grip_r.stl scale=0.001 0.001 0.001
- link link1: geometry collision mesh filename=package://notspot_description/meshes/chain_link1.stl scale=0.001 0.001 0.001; visual mesh filename=package://notspot_description/meshes/chain_link1.stl scale=0.001 0.001 0.001
- link link2: geometry collision mesh filename=package://notspot_description/meshes/chain_link2.stl scale=0.001 0.001 0.001; visual mesh filename=package://notspot_description/meshes/chain_link2.stl scale=0.001 0.001 0.001
- link link3: geometry collision mesh filename=package://notspot_description/meshes/chain_link3.stl scale=0.001 0.001 0.001; visual mesh filename=package://notspot_description/meshes/chain_link3.stl scale=0.001 0.001 0.001
- link link4: geometry collision mesh filename=package://notspot_description/meshes/chain_link4.stl scale=0.001 0.001 0.001; visual mesh filename=package://notspot_description/meshes/chain_link4.stl scale=0.001 0.001 0.001
- link link5: geometry collision mesh filename=package://notspot_description/meshes/chain_link5.stl scale=0.001 0.001 0.001; visual mesh filename=package://notspot_description/meshes/chain_link5.stl scale=0.001 0.001 0.001
- link tray: geometry collision mesh filename=package://notspot_description/meshes/tray.stl scale=0.0004 0.0004 0.0004; visual mesh filename=package://notspot_description/meshes/tray.stl scale=0.0004 0.0004 0.0004
Joints:
- removed joint end_effector_joint
- joint gripper: limit lower=-0.010 upper=0.019 effort=1 velocity=4.8 -> lower=-0.010 upper=0.019 effort=0.3 velocity=1
- joint gripper_sub: limit lower=-0.010 upper=0.019 effort=1 velocity=4.8 -> lower=-0.010 upper=0.019 effort=0.3 velocity=3
- joint joint1: limit lower=${-pi*0.9} upper=${pi*0.9} effort=1 velocity=4.8 -> lower=${-pi*0.9} upper=${pi*0.9} effort=2 velocity=1
- joint joint2: limit lower=${-pi*0.57} upper=${pi*0.5} effort=1 velocity=4.8 -> lower=${-pi*0.57} upper=${pi*0.5} effort=2 velocity=1
- joint joint3: limit lower=${-pi*0.3} upper=${pi*0.44} effort=1 velocity=4.8 -> lower=${-pi*0.3} upper=${pi*0.44} effort=2 velocity=1
- joint joint4: limit lower=${-pi*0.57} upper=${pi*0.65} effort=1 velocity=4.8 -> lower=${-pi*0.57} upper=${pi*0.65} effort=2 velocity=1
